File: 312_project.sch (KiCad schematic (older format))
At the start: 14 parts, among them J1 EMAG_PWM, J2 EMAG_OUT, J3 MOTOR_PWM, J4 LMT_switch, J5 HV_PWR, J6 LV_PWR, J7 MOTOR_OUT, Q1 PN2222A, Q2 IRF540N, U1 TA7267BP

Commit message: added power protection circuit
Parts:
- added U2: RELAY, symbol 312_project-rescue:RELAY
- added U3, U4: Switch, symbol 312_project-rescue:Switch
- U1: symbol symbol:TA7267BP -> 312_project-rescue:TA7267BP-symbol
Connections:
- net labels added: 12V_OUT
- wire segments 36 -> 66
- no-connect marks 0 -> 2
Other:
- note added: "CONNECTORS"
- note added: "ELECTROMAGNET\nCONTROL \nCIRCUIT"
- note added: "MOTOR CONTROL CIRCUIT"
- note added: "PROTECTION \nCIRCUIT"
- moved on the sheet: D1, J1, J2, J3, J4, J5, J6, J7, Q1, Q2, R1, R2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

Commit message: update
Parts:
- added D2: Red LED, symbol Device:LED
- added D3: Green LED, symbol Device:LED
Connections:
- net labels added: 12V_CIRCUIT
- net labels removed: 12V_OUT
- wire segments 66 -> 62
Other:
- note added: "GREEN"
- note added: "RED"
Changed lines of the file:
@@
 P 9375 5000
 F 0 "U3" H 9175 5350 50  0000 L CNN
-F 1 "Switch" H 9375 5350 50  0000 L CNN
+F 1 "Switch" H 9325 5350 50  0000 L CNN
 F 2 "" H 8975 5000 50  0001 C CNN
 F 3 "" H 8975 5000 50  0001 C CNN
@@
 P 9400 6100
 F 0 "U4" H 9200 6450 50  0000 L CNN
-F 1 "Switch" H 9400 6450 50  0000 L CNN
+F 1 "Switch" H 9350 6450 50  0000 L CNN
 F 2 "" H 9000 6100 50  0001 C CNN
 F 3 "" H 9000 6100 50  0001 C CNN
@@
 $EndComp
 Wire Wire Line
-	7350 5925 8825 5925
-Wire Wire Line
-	8825 5925 8825 6100
-Wire Wire Line
 	8825 6100 9100 6100
 Wire Wire Line
@@
 Wire Wire Line
 	8825 4800 9075 4800
-Connection ~ 8825 5925
 Wire Wire Line
 	8825 4800 8825 5425
@@
 Connection ~ 8825 5425
 Wire Wire Line
-	8825 5425 8825 5925
-Wire Wire Line
 	9075 5000 8975 5000
-Wire Wire Line
-	8975 5000 8975 4600
-Wire Wire Line
-	9075 5100 9075 5325
-Wire Wire Line
-	9075 5325 9900 5325
-Wire Wire Line
-	9900 5325 9900 5700
-Wire Wire Line
-	9900 6400 9100 6400
-Wire Wire Line
-	9100 6400 9100 6200
 Wire Wire Line
 	9100 6000 8975 6000
@@
 	8975 5575 7975 5575
 Connection ~ 7975 5575
-Wire Wire Line
-	9900 5700 10225 5700
-Wire Wire Line
-	10225 5700 10225 5825
-Connection ~ 9900 5700
-Wire Wire Line
-	9900 5700 9900 6400
-Wire Wire Line
-	9725 4900 9725 4300
-Wire Wire Line
-	9725 4300 8325 4300
-Wire Wire Line
-	8325 4300 8325 5275
-Wire Wire Line
-	8325 5275 7800 5275
-Wire Wire Line
-	9750 6000 9750 5575
-Wire Wire Line
-	9750 5575 8975 5575
-Connection ~ 8975 5575
 NoConn ~ 9100 5900
 NoConn ~ 9075 4900
@@
 L power:+12V #PWR01
 U 1 1 5D1E96FA
-P 8975 4600
-F 0 "#PWR01" H 8975 4450 50  0001 C CNN
-F 1 "+12V" H 8990 4773 50  0000 C CNN
-F 2 "" H 8975 4600 50  0001 C CNN
-F 3 "" H 8975 4600 50  0001 C CNN
-	1    8975 4600
-	1    0    0    -1
-$EndComp
-$Comp
-L power:GND #PWR02
-U 1 1 5D1EA6DF
-P 10225 5825
-F 0 "#PWR02" H 10225 5575 50  0001 C CNN
-F 1 "GND" H 10230 5652 50  0000 C CNN
-F 2 "" H 10225 5825 50  0001 C CNN
-F 3 "" H 10225 5825 50  0001 C CNN
-	1    10225 5825
+P 9775 5050
+F 0 "#PWR01" H 9775 4900 50  0001 C CNN
+F 1 "+12V" H 9790 5223 50  0000 C CNN
+F 2 "" H 9775 5050 50  0001 C CNN
+F 3 "" H 9775 5050 50  0001 C CNN
+	1    9775 5050
 	1    0    0    -1
 $EndComp
 Text GLabel 8175 5725 2    50   Input ~ 0
-12V_OUT
+12V_CIRCUIT
 Wire Wire Line
 	8175 5725 7975 5725
@@
 Text Notes 1325 1650 0    197  ~ 0
 ELECTROMAGNET\nCONTROL \nCIRCUIT
+$Comp
+L Device:LED D2
+U 1 1 5D1F0DCD
+P 8100 5275
+F 0 "D2" H 8092 5020 50  0000 C CNN
+F 1 "Red LED" H 8092 5111 50  0000 C CNN
+F 2 "" H 8100 5275 50  0001 C CNN
+F 3 "~" H 8100 5275 50  0001 C CNN
+	1    8100 5275
+	-1   0    0    1
+$EndComp
+$Comp
+L Device:LED D3
+U 1 1 5D1F0E46
+P 9300 5575
+F 0 "D3" H 9292 5320 50  0000 C CNN
+F 1 "Green LED" H 9292 5411 50  0000 C CNN
+F 2 "" H 9300 5575 50  0001 C CNN
+F 3 "~" H 9300 5575 50  0001 C CNN
+	1    9300 5575
+	-1   0    0    1
+$EndComp
+Wire Wire Line
+	8975 5575 9150 5575
+Connection ~ 8975 5575
+Wire Wire Line
+	9450 5575 9925 5575
+Wire Wire Line
+	9925 5575 9925 5650
+Wire Wire Line
+	7800 5275 7950 5275
+Wire Wire Line
+	8250 5275 8400 5275
+Wire Wire Line
+	8400 5275 8400 5050
+Wire Wire Line
+	8400 5050 8575 5050
+Wire Wire Line
+	8575 5050 8575 5150
+$Comp
+L power:GND #PWR02
+U 1 1 5D1F7E13
+P 8575 5150
+F 0 "#PWR02" H 8575 4900 50  0001 C CNN
+F 1 "GND" H 8580 4977 50  0000 C CNN
+F 2 "" H 8575 5150 50  0001 C CNN
+F 3 "" H 8575 5150 50  0001 C CNN
+	1    8575 5150
+	1    0    0    -1
+$EndComp
+$Comp
+L power:GND #PWR03
+U 1 1 5D1F8BA5
+P 9925 5650
+F 0 "#PWR03" H 9925 5400 50  0001 C CNN
+F 1 "GND" H 9930 5477 50  0000 C CNN
+F 2 "" H 9925 5650 50  0001 C CNN
+F 3 "" H 9925 5650 50  0001 C CNN
+	1    9925 5650
+	1    0    0    -1
+$EndComp
+Wire Wire Line
+	8975 5000 8975 5125
+Wire Wire Line
+	8975 5125 9775 5125
+Wire Wire Line
+	9775 5125 9775 5050
+Text Notes 9600 4775 0    98   ~ 0
+RED
+Text Notes 9625 6100 0    98   ~ 0
+GREEN
+Wire Wire Line
+	8825 5425 8825 5975
+Wire Wire Line
+	7350 5975 8825 5975
+Connection ~ 8825 5975
+Wire Wire Line
+	8825 5975 8825 6100
 $EndSCHEMATC
